Commit message: resolution bug urdf

File: cdpr/urdf/cube.urdf (robot description, URDF)
Before this commit: robot cdpr, 54 links, 61 joints
Links:
- removed link virt_Ypf0
- removed link virt_Ypf1
- removed link virt_Ypf2
- removed link virt_Ypf3
- removed link virt_Ypf4
- removed link virt_Ypf5
- removed link virt_Ypf6
- removed link virt_Ypf7
Joints:
- removed joint rev_Ypf0
- removed joint rev_Ypf1
- removed joint rev_Ypf2
- removed joint rev_Ypf3
- removed joint rev_Ypf4
- removed joint rev_Ypf5
- removed joint rev_Ypf6
- removed joint rev_Ypf7
- removed joint rev_Zpf0
- removed joint rev_Zpf1
- removed joint rev_Zpf2
- removed joint rev_Zpf3
- removed joint rev_Zpf4
- removed joint rev_Zpf5
- removed joint rev_Zpf6
- removed joint rev_Zpf7
- added joint cable_fixed1: type floating, parent frame_1, child cable0
- added joint cable_fixed2: type floating, parent frame_1, child cable1
- added joint cable_fixed3: type floating, parent frame_1, child cable2
- added joint cable_fixed4: type floating, parent frame_1, child cable3
- added joint cable_fixed5: type floating, parent frame_1, child cable4
- added joint cable_fixed6: type floating, parent frame_1, child cable5
- added joint cable_fixed7: type floating, parent frame_1, child cable6
- added joint cable_fixed8: type floating, parent frame_1, child cable7
- joint joint_cable0: origin xyz=-0.20762000000000003 -0.20762000000000003 0.24372799999999994 rpy=-2.436024 0.575296 -1.353793 -> xyz=0 0 0 rpy=0 0 0
- joint joint_cable1: origin xyz=-0.07723100000000005 0.03693599999999997 0.09066200000000002 rpy=2.754717 0.667932 2.113659 -> xyz=0 0 0 rpy=0 0 0
- joint joint_cable2: origin xyz=-0.06142599999999998 -0.06142599999999998 -0.1507719999999999 rpy=2.754717 -0.360783 -1.499377 -> xyz=0 0 0 rpy=0 0 0
- joint joint_cable3: origin xyz=0.03693599999999997 -0.07723100000000005 0.09066200000000002 rpy=-2.436024 -0.300730 0.780760 -> xyz=0 0 0 rpy=0 0 0
- joint joint_cable4: origin xyz=0.04733199999999993 0.04733199999999993 0.014405 rpy=-1.275355 0.763259 -0.578033 -> xyz=0 0 0 rpy=0 0 0
- joint joint_cable5: origin xyz=0.3567800000000001 -0.17063399999999995 0.108585 rpy=1.004067 1.055080 0.619089 -> xyz=0 0 0 rpy=0 0 0
- joint joint_cable6: origin xyz=-0.566881 -0.566881 0.360742 rpy=1.004067 -0.700803 -0.396004 -> xyz=0 0 0 rpy=0 0 0
- joint joint_cable7: origin xyz=-0.17063399999999995 0.3567800000000001 0.108585 rpy=-1.275355 -0.429106 0.320149 -> xyz=0 0 0 rpy=0 0 0
- joint rev_Xpf0: origin xyz=0 0 0 rpy=-2.436024 0.575296 -1.353793 -> xyz=0 0 0 rpy=0 0 0
- joint rev_Xpf1: origin xyz=0 0 0 rpy=2.754717 0.667932 2.113659 -> xyz=0 0 0 rpy=0 0 0
- joint rev_Xpf2: origin xyz=0 0 0 rpy=2.754717 -0.360783 -1.499377 -> xyz=0 0 0 rpy=0 0 0
- joint rev_Xpf3: origin xyz=0 0 0 rpy=-2.436024 -0.300730 0.780760 -> xyz=0 0 0 rpy=0 0 0
- joint rev_Xpf4: origin xyz=0 0 0 rpy=-1.275355 0.763259 -0.578033 -> xyz=0 0 0 rpy=0 0 0
- joint rev_Xpf5: origin xyz=0 0 0 rpy=1.004067 1.055080 0.619089 -> xyz=0 0 0 rpy=0 0 0
- joint rev_Xpf6: origin xyz=0 0 0 rpy=1.004067 -0.700803 -0.396004 -> xyz=0 0 0 rpy=0 0 0
- joint rev_Xpf7: origin xyz=0 0 0 rpy=-1.275355 -0.429106 0.320149 -> xyz=0 0 0 rpy=0 0 0
- joint rev_Y0: origin xyz=0 0 0 rpy=-2.436024 0.575296 -1.353793 -> xyz=0 0 0 rpy=0 0 0
- joint rev_Y1: origin xyz=0 0 0 rpy=2.754717 0.667932 2.113659 -> xyz=0 0 0 rpy=0 0 0
- joint rev_Y2: origin xyz=0 0 0 rpy=2.754717 -0.360783 -1.499377 -> xyz=0 0 0 rpy=0 0 0
- joint rev_Y3: origin xyz=0 0 0 rpy=-2.436024 -0.300730 0.780760 -> xyz=0 0 0 rpy=0 0 0
- joint rev_Y4: origin xyz=0 0 0 rpy=-1.275355 0.763259 -0.578033 -> xyz=0 0 0 rpy=0 0 0
- joint rev_Y5: origin xyz=0 0 0 rpy=1.004067 1.055080 0.619089 -> xyz=0 0 0 rpy=0 0 0
- joint rev_Y6: origin xyz=0 0 0 rpy=1.004067 -0.700803 -0.396004 -> xyz=0 0 0 rpy=0 0 0
- joint rev_Y7: origin xyz=0 0 0 rpy=-1.275355 -0.429106 0.320149 -> xyz=0 0 0 rpy=0 0 0

File: cdpr/urdf/cube.xacro (robot description, xacro)
@@ -318,6 +318,6 @@
 <xacro:macro name="default_joint_cable" params="num1">
   <joint name="cable_fixed${num1}" type="floating">
-    <child link="frame_1" />
-    <parent link="cable${num1-1}" />
+    <parent link="frame_1" />
+    <child link="cable${num1-1}" />
   </joint>
 </xacro:macro>
@@ -329,4 +329,5 @@
 </xacro:macro>
 <xacro:loop links_qty="10" />
+<xacro:loop2 links_qty="7" />
 <!-- <xacro:loop2 links_qty="7" /> -->
 <!--

File: cdpr/urdf/cube1.xacro (robot description, xacro)
@@ -4,5 +4,4 @@
 	<link name="cable0">
 		<collision>
-			<origin xyz="-0.792380 -0.792380 1.756272" rpy="-2.436024 0.575296 -1.353793"/>
 			<geometry>
 				<cylinder radius="0.005" length="3.4641016151377544"/>
@@ -10,12 +9,11 @@
 		</collision>
 		<visual>
-			<origin xyz="-0.792380 -0.792380 1.756272" rpy="-2.436024 0.575296 -1.353793"/>
-			<geometry>
-				<cylinder radius="0.005" length="3.4641016151377544"/>
-			</geometry>
-			<material name="${cable_color}"/>
-		</visual>
-		<inertial>
-			<origin xyz="-0.792380 -0.792380 1.756272" rpy="-2.436024 0.575296 -1.353793"/>
+			<origin xyz="0 0 0.3815953312159479" rpy="0 0 0"/>
+			<geometry>
+				<cylinder radius="0.005" length="3.4641016151377544"/>
+			</geometry>
+			<material name="${cable_color}"/>
+		</visual>
+		<inertial>
 			<geometry>
 				<cylinder radius="0.005" length="3.4641016151377544"/>
@@ -29,11 +27,12 @@
 			<mass value="0.001"/>
 			<inertia ixx="0.001" ixy="0" ixz="0" iyy="0.001" iyz="0" izz="0.001"/>
-			<origin xyz="-1.000000 -1.000000 2.000000" rpy="-2.436024 0.575296 -1.353793"/>
-		</inertial>
-		<visual>
-			<geometry>
-				<box size="0.1 0.1 0.1"/>
-			</geometry>
-			<material name="${cable_color}"/>
+			<origin xyz="0 0 0" rpy="0 0 0"/>
+		</inertial>
+		<visual>
+			<geometry>
+				<box size="0.1 0.1 0.1"/>
+			</geometry>
+			<material name="${cable_color}"/>
+			<origin xyz="0 0 0" rpy="0 0 0"/>
 		</visual>
 	</link>
@@ -48,10 +47,10 @@
 	<link name="virt_Y0">
 		<inertial>
-			<origin xyz="-1.000000 -1.000000 2.000000" rpy="-2.436024 0.575296 -1.353793"/>
-			<mass value="0.001"/>
-			<inertia ixx="0.001" ixy="0" ixz="0" iyy="0.001" iyz="0" izz="0.001"/>
-			<origin xyz="-1.000000 -1.000000 2.000000" rpy="-2.436024 0.575296 -1.353793"/>
-		</inertial>
-		<visual>
+			<origin xyz="0 0 0" rpy="0 0 0"/>
+			<mass value="0.001"/>
+			<inertia ixx="0.001" ixy="0" ixz="0" iyy="0.001" iyz="0" izz="0.001"/>
+		</inertial>
+		<visual>
+			<origin xyz="0 0 0" rpy="0 0 0"/>
 			<geometry>
 				<box size="0.1 0.1 0.1"/>
@@ -61,5 +60,5 @@
 	</link>
 	<joint name="rev_Y0" type="revolute">
-		<origin xyz="0 0 0" rpy="-2.436024 0.575296 -1.353793"/>
+		<origin xyz="0 0 0" rpy="0 0 0"/>
 		<parent link="virt_X0"/>
 		<child link="virt_Y0"/>
@@ -69,5 +68,5 @@
 	</joint>
 	<joint name="joint_cable0" type="prismatic">
-		<origin xyz="-0.20762000000000003 -0.20762000000000003 0.24372799999999994" rpy="-2.436024 0.575296 -1.353793"/>
+		<origin xyz="0 0 0" rpy="0 0 0"/>
 		<parent link="virt_Y0"/>
 		<child link="cable0"/>
@@ -75,4 +74,5 @@
 		<limit lower="-1.7320508075688772" upper="1.7320508075688772" effort="10000" velocity="0.25"/>
 		<limit damping="0.1"/>
+		<origin xyz="0 0 0" rpy="-2.436024 0.575296 -1.353793"/>
 	</joint>
 	<link name="virt_Xpf0">
@@ -88,13 +88,8 @@
 			</geometry>
 			<material name="${cable_color}"/>
-			<origin xyz="0.150000 0.150000 0.650000" rpy="-2.436024 0.575296 -1.353793"/>
-			<geometry>
-				<box size="0.1 0.1 0.1"/>
-			</geometry>
-			<material name="${cable_color}"/>
 		</visual>
 	</link>
 	<joint name="rev_Xpf0" type="revolute">
-		<origin xyz="0 0 0" rpy="-2.436024 0.575296 -1.353793"/>
+		<origin xyz="0 0 0" rpy="0 0 0"/>
 		<parent link="platform"/>
 		<child link="virt_Xpf0"/>
@@ -103,30 +98,6 @@
 		<limit damping="0.1"/>
 	</joint>
-	<link name="virt_Ypf0">
-		<inertial>
-			<origin xyz="0.150000 0.150000 0.650000" rpy="-2.436024 0.575296 -1.353793"/>
-			<mass value="0.001"/>
-			<inertia ixx="0.001" ixy="0" ixz="0" iyy="0.001" iyz="0" izz="0.001"/>
-		</inertial>
-	</link>
-	<joint name="rev_Ypf0" type="revolute">
-		<origin xyz="0 0 0" rpy="-2.436024 0.575296 -1.353793"/>
-		<parent link="virt_Xpf0"/>
-		<child link="virt_Ypf0"/>
-		<axis xyz="0 1 0"/>
-		<limit effort="10000" velocity="0.25"/>
-		<limit damping="0.1"/>
-	</joint>
-	<joint name="rev_Zpf0" type="revolute">
-		<origin xyz="0.150000 0.150000 0.650000" rpy="-2.436024 0.575296 -1.353793"/>
-		<parent link="cable0"/>
-		<child link="virt_Ypf0"/>
-		<axis xyz="0 0 1"/>
-		<limit effort="10000" velocity="0.25"/>
-		<limit damping="0.1"/>
-	</joint>
 	<link name="cable1">
 		<collision>
-			<origin xyz="-0.922769 0.963064 1.909338" rpy="2.754717 0.667932 2.113659"/>
 			<geometry>
 				<cylinder radius="0.005" length="3.4641016151377544"/>
@@ -134,12 +105,11 @@
 		</collision>
 		<visual>
-			<origin xyz="-0.922769 0.963064 1.909338" rpy="2.754717 0.667932 2.113659"/>
-			<geometry>
-				<cylinder radius="0.005" length="3.4641016151377544"/>
-			</geometry>
-			<material name="${cable_color}"/>
-		</visual>
-		<inertial>
-			<origin xyz="-0.922769 0.963064 1.909338" rpy="2.754717 0.667932 2.113659"/>
+			<origin xyz="0 0 0.1246936551938369" rpy="0 0 0"/>
+			<geometry>
+				<cylinder radius="0.005" length="3.4641016151377544"/>
+			</geometry>
+			<material name="${cable_color}"/>
+		</visual>
+		<inertial>
 			<geometry>
 				<cylinder radius="0.005" length="3.4641016151377544"/>
@@ -153,11 +123,12 @@
 			<mass value="0.001"/>
 			<inertia ixx="0.001" ixy="0" ixz="0" iyy="0.001" iyz="0" izz="0.001"/>
-			<origin xyz="-1.000000 1.000000 2.000000" rpy="2.754717 0.667932 2.113659"/>
-		</inertial>
-		<visual>
-			<geometry>
-				<box size="0.1 0.1 0.1"/>
-			</geometry>
-			<material name="${cable_color}"/>
+			<origin xyz="0 0 0" rpy="0 0 0"/>
+		</inertial>
+		<visual>
+			<geometry>
+				<box size="0.1 0.1 0.1"/>
+			</geometry>
+			<material name="${cable_color}"/>
+			<origin xyz="0 0 0" rpy="0 0 0"/>
 		</visual>
 	</link>
@@ -172,10 +143,10 @@
 	<link name="virt_Y1">
 		<inertial>
-			<origin xyz="-1.000000 1.000000 2.000000" rpy="2.754717 0.667932 2.113659"/>
-			<mass value="0.001"/>
-			<inertia ixx="0.001" ixy="0" ixz="0" iyy="0.001" iyz="0" izz="0.001"/>
-			<origin xyz="-1.000000 1.000000 2.000000" rpy="2.754717 0.667932 2.113659"/>
-		</inertial>
-		<visual>
+			<origin xyz="0 0 0" rpy="0 0 0"/>
+			<mass value="0.001"/>
+			<inertia ixx="0.001" ixy="0" ixz="0" iyy="0.001" iyz="0" izz="0.001"/>
+		</inertial>
+		<visual>
+			<origin xyz="0 0 0" rpy="0 0 0"/>
 			<geometry>
 				<box size="0.1 0.1 0.1"/>
@@ -185,5 +156,5 @@
 	</link>
 	<joint name="rev_Y1" type="revolute">
-		<origin xyz="0 0 0" rpy="2.754717 0.667932 2.113659"/>
+		<origin xyz="0 0 0" rpy="0 0 0"/>
 		<parent link="virt_X1"/>
 		<child link="virt_Y1"/>
@@ -193,5 +164,5 @@
 	</joint>
 	<joint name="joint_cable1" type="prismatic">
-		<origin xyz="-0.07723100000000005 0.03693599999999997 0.09066200000000002" rpy="2.754717 0.667932 2.113659"/>
+		<origin xyz="0 0 0" rpy="0 0 0"/>
 		<parent link="virt_Y1"/>
 		<child link="cable1"/>
@@ -199,4 +170,5 @@
 		<limit lower="-1.7320508075688772" upper="1.7320508075688772" effort="10000" velocity="0.25"/>
 		<limit damping="0.1"/>
+		<origin xyz="0 0 0" rpy="2.754717 0.667932 2.113659"/>
 	</joint>
 	<link name="virt_Xpf1">
@@ -212,13 +184,8 @@
 			</geometry>
 			<material name="${cable_color}"/>
-			<origin xyz="0.150000 0.450000 0.650000" rpy="2.754717 0.667932 2.113659"/>
-			<geometry>
-				<box size="0.1 0.1 0.1"/>
-			</geometry>
-			<material name="${cable_color}"/>
 		</visual>
 	</link>
 	<joint name="rev_Xpf1" type="revolute">
-		<origin xyz="0 0 0" rpy="2.754717 0.667932 2.113659"/>
+		<origin xyz="0 0 0" rpy="0 0 0"/>
 		<parent link="platform"/>
 		<child link="virt_Xpf1"/>
@@ -227,30 +194,6 @@
 		<limit damping="0.1"/>
 	</joint>
-	<link name="virt_Ypf1">
-		<inertial>
-			<origin xyz="0.150000 0.450000 0.650000" rpy="2.754717 0.667932 2.113659"/>
-			<mass value="0.001"/>
-			<inertia ixx="0.001" ixy="0" ixz="0" iyy="0.001" iyz="0" izz="0.001"/>
-		</inertial>
-	</link>
-	<joint name="rev_Ypf1" type="revolute">
-		<origin xyz="0 0 0" rpy="2.754717 0.667932 2.113659"/>
-		<parent link="virt_Xpf1"/>
-		<child link="virt_Ypf1"/>
-		<axis xyz="0 1 0"/>
-		<limit effort="10000" velocity="0.25"/>
-		<limit damping="0.1"/>
-	</joint>
-	<joint name="rev_Zpf1" type="revolute">
-		<origin xyz="0.150000 0.450000 0.650000" rpy="2.754717 0.667932 2.113659"/>
-		<parent link="cable1"/>
-		<child link="virt_Ypf1"/>
-		<axis xyz="0 0 1"/>
-		<limit effort="10000" velocity="0.25"/>
-		<limit damping="0.1"/>
-	</joint>
 	<link name="cable2">
 		<collision>
-			<origin xyz="1.061426 1.061426 2.150772" rpy="2.754717 -0.360783 -1.499377"/>
 			<geometry>
 				<cylinder radius="0.005" length="3.4641016151377544"/>
@@ -258,12 +201,11 @@
 		</collision>
 		<visual>
-			<origin xyz="1.061426 1.061426 2.150772" rpy="2.754717 -0.360783 -1.499377"/>
-			<geometry>
-				<cylinder radius="0.005" length="3.4641016151377544"/>
-			</geometry>
-			<material name="${cable_color}"/>
-		</visual>
-		<inertial>
-			<origin xyz="1.061426 1.061426 2.150772" rpy="2.754717 -0.360783 -1.499377"/>
+			<origin xyz="0 0 -0.17400716248058878" rpy="0 0 0"/>
+			<geometry>
+				<cylinder radius="0.005" length="3.4641016151377544"/>
+			</geometry>
+			<material name="${cable_color}"/>
+		</visual>
+		<inertial>
 			<geometry>
 				<cylinder radius="0.005" length="3.4641016151377544"/>
@@ -277,11 +219,12 @@
 			<mass value="0.001"/>
 			<inertia ixx="0.001" ixy="0" ixz="0" iyy="0.001" iyz="0" izz="0.001"/>
-			<origin xyz="1.000000 1.000000 2.000000" rpy="2.754717 -0.360783 -1.499377"/>
-		</inertial>
-		<visual>
-			<geometry>
-				<box size="0.1 0.1 0.1"/>
-			</geometry>
-			<material name="${cable_color}"/>
+			<origin xyz="0 0 0" rpy="0 0 0"/>
+		</inertial>
+		<visual>
+			<geometry>
+				<box size="0.1 0.1 0.1"/>
+			</geometry>
+			<material name="${cable_color}"/>
+			<origin xyz="0 0 0" rpy="0 0 0"/>
 		</visual>
 	</link>
@@ -296,10 +239,10 @@
 	<link name="virt_Y2">
 		<inertial>
-			<origin xyz="1.000000 1.000000 2.000000" rpy="2.754717 -0.360783 -1.499377"/>
-			<mass value="0.001"/>
-			<inertia ixx="0.001" ixy="0" ixz="0" iyy="0.001" iyz="0" izz="0.001"/>
-			<origin xyz="1.000000 1.000000 2.000000" rpy="2.754717 -0.360783 -1.499377"/>
-		</inertial>
-		<visual>
+			<origin xyz="0 0 0" rpy="0 0 0"/>
+			<mass value="0.001"/>
+			<inertia ixx="0.001" ixy="0" ixz="0" iyy="0.001" iyz="0" izz="0.001"/>
+		</inertial>
+		<visual>
+			<origin xyz="0 0 0" rpy="0 0 0"/>
 			<geometry>
 				<box size="0.1 0.1 0.1"/>
@@ -309,5 +252,5 @@
 	</link>
 	<joint name="rev_Y2" type="revolute">
-		<origin xyz="0 0 0" rpy="2.754717 -0.360783 -1.499377"/>
+		<origin xyz="0 0 0" rpy="0 0 0"/>
 		<parent link="virt_X2"/>
 		<child link="virt_Y2"/>
@@ -317,5 +260,5 @@
 	</joint>
 	<joint name="joint_cable2" type="prismatic">
-		<origin xyz="-0.06142599999999998 -0.06142599999999998 -0.1507719999999999" rpy="2.754717 -0.360783 -1.499377"/>
+		<origin xyz="0 0 0" rpy="0 0 0"/>
 		<parent link="virt_Y2"/>
 		<child link="cable2"/>
@@ -323,4 +266,5 @@
 		<limit lower="-1.7320508075688772" upper="1.7320508075688772" effort="10000" velocity="0.25"/>
 		<limit damping="0.1"/>
+		<origin xyz="0 0 0" rpy="2.754717 -0.360783 -1.499377"/>
 	</joint>
 	<link name="virt_Xpf2">
@@ -336,13 +280,8 @@
 			</geometry>
 			<material name="${cable_color}"/>
-			<origin xyz="0.450000 0.450000 0.650000" rpy="2.754717 -0.360783 -1.499377"/>
-			<geometry>
-				<box size="0.1 0.1 0.1"/>
-			</geometry>
-			<material name="${cable_color}"/>
 		</visual>
 	</link>
 	<joint name="rev_Xpf2" type="revolute">
-		<origin xyz="0 0 0" rpy="2.754717 -0.360783 -1.499377"/>
+		<origin xyz="0 0 0" rpy="0 0 0"/>
 		<parent link="platform"/>
 		<child link="virt_Xpf2"/>
@@ -351,30 +290,6 @@
 		<limit damping="0.1"/>
 	</joint>
-	<link name="virt_Ypf2">
-		<inertial>
-			<origin xyz="0.450000 0.450000 0.650000" rpy="2.754717 -0.360783 -1.499377"/>
-			<mass value="0.001"/>
-			<inertia ixx="0.001" ixy="0" ixz="0" iyy="0.001" iyz="0" izz="0.001"/>
-		</inertial>
-	</link>
-	<joint name="rev_Ypf2" type="revolute">
-		<origin xyz="0 0 0" rpy="2.754717 -0.360783 -1.499377"/>
-		<parent link="virt_Xpf2"/>
-		<child link="virt_Ypf2"/>
-		<axis xyz="0 1 0"/>
-		<limit effort="10000" velocity="0.25"/>
-		<limit damping="0.1"/>
-	</joint>
-	<joint name="rev_Zpf2" type="revolute">
-		<origin xyz="0.450000 0.450000 0.650000" rpy="2.754717 -0.360783 -1.499377"/>
-		<parent link="cable2"/>
-		<child link="virt_Ypf2"/>
-		<axis xyz="0 0 1"/>
-		<limit effort="10000" velocity="0.25"/>
-		<limit damping="0.1"/>
-	</joint>
 	<link name="cable3">
 		<collision>
-			<origin xyz="0.963064 -0.922769 1.909338" rpy="-2.436024 -0.300730 0.780760"/>
 			<geometry>
 				<cylinder radius="0.005" length="3.4641016151377544"/>
@@ -382,12 +297,11 @@
 		</collision>
 		<visual>
-			<origin xyz="0.963064 -0.922769 1.909338" rpy="-2.436024 -0.300730 0.780760"/>
-			<geometry>
-				<cylinder radius="0.005" length="3.4641016151377544"/>
-			</geometry>
-			<material name="${cable_color}"/>
-		</visual>
-		<inertial>
-			<origin xyz="0.963064 -0.922769 1.909338" rpy="-2.436024 -0.300730 0.780760"/>
+			<origin xyz="0 0 0.1246936551938369" rpy="0 0 0"/>
+			<geometry>
+				<cylinder radius="0.005" length="3.4641016151377544"/>
+			</geometry>
+			<material name="${cable_color}"/>
+		</visual>
+		<inertial>
 			<geometry>
 				<cylinder radius="0.005" length="3.4641016151377544"/>
@@ -401,11 +315,12 @@
 			<mass value="0.001"/>
 			<inertia ixx="0.001" ixy="0" ixz="0" iyy="0.001" iyz="0" izz="0.001"/>
-			<origin xyz="1.000000 -1.000000 2.000000" rpy="-2.436024 -0.300730 0.780760"/>
-		</inertial>
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