Commit message: fin du projet

File: cdpr/urdf/cube.urdf (robot description, URDF)
Before this commit: robot cdpr, 46 links, 53 joints
Links:
- added link virt_Ypf0, mass 0.001
- added link virt_Ypf1, mass 0.001
- added link virt_Ypf2, mass 0.001
- added link virt_Ypf3, mass 0.001
- added link virt_Ypf4, mass 0.001
- added link virt_Ypf5, mass 0.001
- added link virt_Ypf6, mass 0.001
- added link virt_Ypf7, mass 0.001
Joints:
- removed joint cable_fixed1
- removed joint cable_fixed2
- removed joint cable_fixed3
- removed joint cable_fixed4
- removed joint cable_fixed5
- removed joint cable_fixed6
- removed joint cable_fixed7
- removed joint cable_fixed8
- removed joint float
- added joint float_platform: type floating, parent world, child platform
- added joint rev_Zpf0: type revolute, parent cable0, child virt_Ypf0, origin xyz=0 0 1.7320508075688772 rpy=0 0 0, axis 0 0 1, limit effort=10000 velocity=0.25
- added joint rev_Zpf1: type revolute, parent cable1, child virt_Ypf1, origin xyz=0 0 1.7320508075688772 rpy=0 0 0, axis 0 0 1, limit effort=10000 velocity=0.25
- added joint rev_Zpf2: type revolute, parent cable2, child virt_Ypf2, origin xyz=0 0 1.7320508075688772 rpy=0 0 0, axis 0 0 1, limit effort=10000 velocity=0.25
- added joint rev_Zpf3: type revolute, parent cable3, child virt_Ypf3, origin xyz=0 0 1.7320508075688772 rpy=0 0 0, axis 0 0 1, limit effort=10000 velocity=0.25
- added joint rev_Zpf4: type revolute, parent cable4, child virt_Ypf4, origin xyz=0 0 1.7320508075688772 rpy=0 0 0, axis 0 0 1, limit effort=10000 velocity=0.25
- added joint rev_Zpf5: type revolute, parent cable5, child virt_Ypf5, origin xyz=0 0 1.7320508075688772 rpy=0 0 0, axis 0 0 1, limit effort=10000 velocity=0.25
- added joint rev_Zpf6: type revolute, parent cable6, child virt_Ypf6, origin xyz=0 0 1.7320508075688772 rpy=0 0 0, axis 0 0 1, limit effort=10000 velocity=0.25
- added joint rev_Zpf7: type revolute, parent cable7, child virt_Ypf7, origin xyz=0 0 1.7320508075688772 rpy=0 0 0, axis 0 0 1, limit effort=10000 velocity=0.25

File: cdpr/urdf/cube.xacro (robot description, xacro)
@@ -2,9 +2,11 @@
 <!-- Revolute-Revolute Manipulator -->
 <robot name="cdpr" xmlns:xacro="http://www.ros.org/wiki/xacro">
+<!-- Ce code permet de générer le cadre du robot, les liaisons entre les parties du cadre et la plateforme-->
+<!-- Bien faire gaffe à repercuter les valeurs des paramètres changés ici sur cube1.yaml-->
   <!-- Constants for robot dimensions -->
   <xacro:property name="PI" value="3.1415926535897931" />
-  <xacro:property name="cable_mass" value="0.001" /> <!-- arbitrary value for mass -->
+  <xacro:property name="cable_mass" value="0.001" />
   <xacro:property name="cable_radius" value="0.001" />
-  <xacro:property name="frame_color" value="orange" /> <!-- Square dimensions (widthxwidth) of beams -->
+  <xacro:property name="frame_color" value="orange" /> <!-- les couleurs ne fonctionnent pas en fait, que sur urdf viewer -->
   <xacro:property name="frame_lower" value="1.0 1.0 0" />
   <xacro:property name="frame_radius" value="0.02" />
@@ -21,13 +23,6 @@
   <xacro:property name="platform_iaa" value="0.33" /> <!-- ixx iyy izz-->
   <xacro:property name="platform_iab" value="0" />
-  <xacro:property name="mass" value="1" /> <!-- arbitrary value for mass -->
-  <xacro:property name="width" value="0.1" /> <!-- Square dimensions (widthxwidth) of beams -->
-  <xacro:property name="height1" value="2" /> <!-- Link 1 -->
-  <xacro:property name="height2" value="1" /> <!-- Link 2 -->
-  <xacro:property name="height3" value="1" /> <!-- Link 3 -->
-  <xacro:property name="camera_link" value="0.05" /> <!-- Size of square 'camera' box -->
-  <xacro:property name="axel_offset" value="0.05" />
-  <!-- Import all Gazebo-customization elements, including Gazebo colors -->
-  <!--<xacro:include filename="$(find cdpr)/urdf/cube.gazebo" /> -->
+  <!-- Import all Gazebo-customization elements, including Gazebo colors(au cas ca marcherait un jour) -->
+ <xacro:include filename="$(find cdpr)/urdf/cube.gazebo" />
   <!-- Import Rviz colors -->
   <xacro:include filename="$(find cdpr)/urdf/materials.xacro" />
@@ -39,8 +34,47 @@
     <child link="frame_1" />
   </joint>
-  <joint name="float" type="floating">
+  <!-- le float n'existe pas en sdf et cette liaison sera transformée en fixed dans gazebo -->
+  <!-- Il faut trouver une solution pour le rendre mobile en selectionnant un jeu de liaison qui le lie à world -->
+  <joint name="float_platform" type="floating">
     <parent link="world" />
-    <child link="platform"/>
-  </joint>
+    <child link="platform" />
+  </joint>
+<!--
+  <link name="virt_Xl">
+		<inertial>
+			<origin xyz="0 0 0" rpy="0 0 0"/>
+			<mass value="0.001"/>
+			<inertia ixx="0.001" ixy="0" ixz="0" iyy="0.001" iyz="0" izz="0.001"/>
+		</inertial>
+	</link>
+  <joint name="prism_1" type="prismatic">
+    <origin xyz="0 0 0" rpy="0 0 0"/>
+    <parent link="virt_X1" />
+    <child link="platform" />
+    <limit lower="-2" upper="2" effort="10000" velocity="1"/>
+    <axis xyz="1 0 0"/>
+  </joint>
+  <link name="virt_Yl">
+		<inertial>
+			<origin xyz="0 0 0" rpy="0 0 0"/>
+			<mass value="0.001"/>
+			<inertia ixx="0.001" ixy="0" ixz="0" iyy="0.001" iyz="0" izz="0.001"/>
+		</inertial>
+	</link>
+  <joint name="prism2" type="prismatic">
+    <origin xyz="0 0 0" rpy="0 0 0"/>
+    <parent link="virt_X1" />
+    <child link="virt_Y1" />
+    <limit lower="-2" upper="2" effort="10000" velocity="1"/>
+    <axis xyz="1 0 0"/>
+  </joint>
+  <joint name="prism3" type="prismatic">
+    <origin xyz="0 0 0" rpy="0 0 0"/>
+    <parent link="world" />
+    <child link="virt_Y1" />
+    <limit lower="-2" upper="2" effort="10000" velocity="1"/>
+    <axis xyz="0 0 1"/>
+  </joint>
+-->
   <!-- Base Link -->
   <link name="frame_1">
@@ -304,5 +338,5 @@
     </inertial>
   </link>
-<xacro:macro name="default_joint" params="num1 num2">
+<xacro:macro name="default_joint" params="num1 num2"> <!-- définit une macro de liaison entre les parties du cube -->
   <joint name="fixed${num1}" type="fixed">
     <parent link="frame_${num2}" />
@@ -310,5 +344,5 @@
   </joint>
 </xacro:macro>
-<xacro:macro name="loop" params="links_qty">
+<xacro:macro name="loop" params="links_qty"> <!-- permet d'executer la macro en boucle -->
   <xacro:default_joint num1="${links_qty+2}" num2="${links_qty+1}"/>
     <xacro:if value="${links_qty}">
@@ -316,4 +350,5 @@
     </xacro:if>
 </xacro:macro>
+<!-- Ne sert plus mais permettait de fixer les cables au cadre pour tester les liaisons -->
 <xacro:macro name="default_joint_cable" params="num1">
   <joint name="cable_fixed${num1}" type="floating">
@@ -328,117 +363,5 @@
     </xacro:if>
 </xacro:macro>
-<xacro:loop links_qty="10" />
-<xacro:loop2 links_qty="7" />
+<xacro:loop links_qty="10" /> <!-- execute la macro -->
 <!-- <xacro:loop2 links_qty="7" /> -->
-<!--
-<joint name="platform_frame_fixed$" type="fixed">
-  <parent link="frame_1" />
-  <child link="platform" />
-</joint> -->
-  <!-- Camera -->
-  <!--
-  <link name="camera_link">
-    <collision>
-      <origin xyz="0 0 0" rpy="0 0 0" />
-      <geometry>
-        <box size="${camera_link} ${camera_link} ${camera_link}" />
-      </geometry>
-    </collision>
-    <visual>
-      <origin xyz="0 0 0" rpy="0 0 0" />
-      <geometry>
-        <box size="${camera_link} ${camera_link} ${camera_link}" />
-      </geometry>
-      <material name="red" />
-    </visual>
-    <inertial>
-      <mass value="1e-5" />
-      <origin xyz="0 0 0" rpy="0 0 0" />
-      <inertia ixx="1e-6" ixy="0" ixz="0" iyy="1e-6" iyz="0" izz="1e-6" />
-    </inertial>
-  </link>
-  <link name="camera_link_optical"></link>
-  -->
-  <!--
-  <transmission name="lift_transmission">
-    <type>transmission_interface/SimpleTransmission</type>
-    <joint name="cable0">
-        <hardwareInterface>PositionJointInterface</hardwareInterface>
-    </joint>
-    <actuator name="lift_motor_0">
-        <hardwareInterface>PositionJointInterface</hardwareInterface>
-        <mechanicalReduction>1</mechanicalReduction>
-    </actuator>
-  </transmission>
-  <transmission name="lift_transmission_1">
-    <type>transmission_interface/SimpleTransmission</type>
-    <joint name="cable1">
-        <hardwareInterface>PositionJointInterface</hardwareInterface>
-    </joint>
-    <actuator name="lift_motor_1">
-        <hardwareInterface>PositionJointInterface</hardwareInterface>
-        <mechanicalReduction>1</mechanicalReduction>
-    </actuator>
-  </transmission>
-  <transmission name="lift_transmission_2">
-    <type>transmission_interface/SimpleTransmission</type>
-    <joint name="cable2">
-        <hardwareInterface>PositionJointInterface</hardwareInterface>
-    </joint>
-    <actuator name="lift_motor_2">
-        <hardwareInterface>PositionJointInterface</hardwareInterface>
-        <mechanicalReduction>1</mechanicalReduction>
-    </actuator>
-  </transmission>
-  <transmission name="lift_transmission_3">
-    <type>transmission_interface/SimpleTransmission</type>
-    <joint name="cable3">
-        <hardwareInterface>PositionJointInterface</hardwareInterface>
-    </joint>
-    <actuator name="lift_motor_3">
-        <hardwareInterface>PositionJointInterface</hardwareInterface>
-        <mechanicalReduction>1</mechanicalReduction>
-    </actuator>
-  </transmission>
-  <transmission name="lift_transmission_4">
-    <type>transmission_interface/SimpleTransmission</type>
-    <joint name="cable4">
-        <hardwareInterface>PositionJointInterface</hardwareInterface>
-    </joint>
-    <actuator name="lift_motor_4">
-        <hardwareInterface>PositionJointInterface</hardwareInterface>
-        <mechanicalReduction>1</mechanicalReduction>
-    </actuator>
-  </transmission>
-  <transmission name="lift_transmission_5">
-    <type>transmission_interface/SimpleTransmission</type>
-    <joint name="cable5">
-        <hardwareInterface>PositionJointInterface</hardwareInterface>
-    </joint>
-    <actuator name="lift_motor_5">
-        <hardwareInterface>PositionJointInterface</hardwareInterface>
-        <mechanicalReduction>1</mechanicalReduction>
-    </actuator>
-  </transmission>
-  <transmission name="lift_transmission_6">
-    <type>transmission_interface/SimpleTransmission</type>
-    <joint name="cable6">
-        <hardwareInterface>PositionJointInterface</hardwareInterface>
-    </joint>
-    <actuator name="lift_motor_6">
-        <hardwareInterface>PositionJointInterface</hardwareInterface>
-        <mechanicalReduction>1</mechanicalReduction>
-    </actuator>
-  </transmission>
-  <transmission name="lift_transmission_7">
-    <type>transmission_interface/SimpleTransmission</type>
-    <joint name="cable7">
-        <hardwareInterface>PositionJointInterface</hardwareInterface>
-    </joint>
-    <actuator name="lift_motor_7">
-        <hardwareInterface>PositionJointInterface</hardwareInterface>
-        <mechanicalReduction>1</mechanicalReduction>
-    </actuator>
-  </transmission>
--->
 </robot>

File: cdpr/urdf/cube1.xacro (robot description, xacro)
@@ -4,4 +4,5 @@
 	<link name="cable0">
 		<collision>
+			<origin xyz="0 0 0.3815953312159479" rpy="0 0 0"/>
 			<geometry>
 				<cylinder radius="0.005" length="3.4641016151377544"/>
@@ -16,4 +17,5 @@
 		</visual>
 		<inertial>
+			<origin xyz="0 0 0.3815953312159479" rpy="0 0 0"/>
 			<geometry>
 				<cylinder radius="0.005" length="3.4641016151377544"/>
@@ -88,4 +90,9 @@
 			</geometry>
 			<material name="${cable_color}"/>
+			<origin xyz="0.150000 0.150000 0.650000" rpy="-2.436024 0.575296 -1.353793"/>
+			<geometry>
+				<box size="0.1 0.1 0.1"/>
+			</geometry>
+			<material name="${cable_color}"/>
 		</visual>
 	</link>
@@ -98,6 +105,45 @@
 		<limit damping="0.1"/>
 	</joint>
+	<link name="virt_Ypf0">
+		<inertial>
+			<origin xyz="0 0 0" rpy="0 0 0"/>
+			<mass value="0.001"/>
+			<inertia ixx="0.001" ixy="0" ixz="0" iyy="0.001" iyz="0" izz="0.001"/>
+		</inertial>
+	</link>
+	<joint name="rev_Zpf0" type="revolute">
+		<origin xyz="0 0 1.7320508075688772" rpy="0 0 0"/>
+		<parent link="cable0"/>
+		<child link="virt_Ypf0"/>
+		<axis xyz="0 0 1"/>
+		<limit effort="10000" velocity="0.25"/>
+		<limit damping="0.1"/>
+	</joint>
+	<gazebo>
+		<joint name="rev_Ypf0" type="revolute">
+			<pose>0 0 0 -2.436024 0.575296 -1.353793</pose>
+			<parent>virt_Xpf0</parent>
+			<child>virt_Ypf0</child>
+			<axis>
+				<xyz>0 1 0</xyz>
+				<limit>
+					<effort>10000</effort>
+					<velocity>0.25</velocity>
+				</limit>
+				<dynamics>
+					<damping>0.1</damping>
+				</dynamics>
+			</axis>
+		</joint>
+	</gazebo>
+	<gazebo reference="cable0">
+		<material>Gazebo/Red</material>
+	</gazebo>
+	<gazebo reference="cable0">
+		<material>Gazebo/Red</material>
+	</gazebo>
 	<link name="cable1">
 		<collision>
+			<origin xyz="0 0 0.1246936551938369" rpy="0 0 0"/>
 			<geometry>
 				<cylinder radius="0.005" length="3.4641016151377544"/>
@@ -112,4 +158,5 @@
 		</visual>
 		<inertial>
+			<origin xyz="0 0 0.1246936551938369" rpy="0 0 0"/>
 			<geometry>
 				<cylinder radius="0.005" length="3.4641016151377544"/>
@@ -184,4 +231,9 @@
 			</geometry>
 			<material name="${cable_color}"/>
+			<origin xyz="0.150000 0.450000 0.650000" rpy="2.754717 0.667932 2.113659"/>
+			<geometry>
+				<box size="0.1 0.1 0.1"/>
+			</geometry>
+			<material name="${cable_color}"/>
 		</visual>
 	</link>
@@ -194,6 +246,45 @@
 		<limit damping="0.1"/>
 	</joint>
+	<link name="virt_Ypf1">
+		<inertial>
+			<origin xyz="0 0 0" rpy="0 0 0"/>
+			<mass value="0.001"/>
+			<inertia ixx="0.001" ixy="0" ixz="0" iyy="0.001" iyz="0" izz="0.001"/>
+		</inertial>
+	</link>
+	<joint name="rev_Zpf1" type="revolute">
+		<origin xyz="0 0 1.7320508075688772" rpy="0 0 0"/>
+		<parent link="cable1"/>
+		<child link="virt_Ypf1"/>
+		<axis xyz="0 0 1"/>
+		<limit effort="10000" velocity="0.25"/>
+		<limit damping="0.1"/>
+	</joint>
+	<gazebo>
+		<joint name="rev_Ypf1" type="revolute">
+			<pose>0 0 0 2.754717 0.667932 2.113659</pose>
+			<parent>virt_Xpf1</parent>
+			<child>virt_Ypf1</child>
+			<axis>
+				<xyz>0 1 0</xyz>
+				<limit>
+					<effort>10000</effort>
+					<velocity>0.25</velocity>
+				</limit>
+				<dynamics>
+					<damping>0.1</damping>
+				</dynamics>
+			</axis>
+		</joint>
+	</gazebo>
+	<gazebo reference="cable1">
+		<material>Gazebo/Red</material>
+	</gazebo>
+	<gazebo reference="cable1">
+		<material>Gazebo/Red</material>
+	</gazebo>
 	<link name="cable2">
 		<collision>
+			<origin xyz="0 0 -0.17400716248058878" rpy="0 0 0"/>
 			<geometry>
 				<cylinder radius="0.005" length="3.4641016151377544"/>
@@ -208,4 +299,5 @@
 		</visual>
 		<inertial>
+			<origin xyz="0 0 -0.17400716248058878" rpy="0 0 0"/>
 			<geometry>
 				<cylinder radius="0.005" length="3.4641016151377544"/>
@@ -280,4 +372,9 @@
 			</geometry>
 			<material name="${cable_color}"/>
+			<origin xyz="0.450000 0.450000 0.650000" rpy="2.754717 -0.360783 -1.499377"/>
+			<geometry>
+				<box size="0.1 0.1 0.1"/>
+			</geometry>
+			<material name="${cable_color}"/>
 		</visual>
 	</link>
@@ -290,6 +387,45 @@
 		<limit damping="0.1"/>
 	</joint>
+	<link name="virt_Ypf2">
+		<inertial>
+			<origin xyz="0 0 0" rpy="0 0 0"/>
+			<mass value="0.001"/>
+			<inertia ixx="0.001" ixy="0" ixz="0" iyy="0.001" iyz="0" izz="0.001"/>
+		</inertial>
+	</link>
+	<joint name="rev_Zpf2" type="revolute">
+		<origin xyz="0 0 1.7320508075688772" rpy="0 0 0"/>
+		<parent link="cable2"/>
+		<child link="virt_Ypf2"/>
+		<axis xyz="0 0 1"/>
+		<limit effort="10000" velocity="0.25"/>
+		<limit damping="0.1"/>
+	</joint>
+	<gazebo>
+		<joint name="rev_Ypf2" type="revolute">
+			<pose>0 0 0 2.754717 -0.360783 -1.499377</pose>
+			<parent>virt_Xpf2</parent>
+			<child>virt_Ypf2</child>
+			<axis>
+				<xyz>0 1 0</xyz>
+				<limit>
+					<effort>10000</effort>
+					<velocity>0.25</velocity>
+				</limit>
+				<dynamics>
+					<damping>0.1</damping>
+				</dynamics>
+			</axis>
+		</joint>
+	</gazebo>
+	<gazebo reference="cable2">
+		<material>Gazebo/Red</material>
+	</gazebo>
+	<gazebo reference="cable2">
+		<material>Gazebo/Red</material>
+	</gazebo>
 	<link name="cable3">
 		<collision>
+			<origin xyz="0 0 0.1246936551938369" rpy="0 0 0"/>
 			<geometry>
 				<cylinder radius="0.005" length="3.4641016151377544"/>
@@ -304,4 +440,5 @@
 		</visual>
 		<inertial>
+			<origin xyz="0 0 0.1246936551938369" rpy="0 0 0"/>
 			<geometry>
 				<cylinder radius="0.005" length="3.4641016151377544"/>
@@ -376,4 +513,9 @@
 			</geometry>
 			<material name="${cable_color}"/>
+			<origin xyz="0.450000 0.150000 0.650000" rpy="-2.436024 -0.300730 0.780760"/>
+			<geometry>
+				<box size="0.1 0.1 0.1"/>
+			</geometry>
+			<material name="${cable_color}"/>
 		</visual>
 	</link>
@@ -386,6 +528,45 @@
 		<limit damping="0.1"/>
 	</joint>
+	<link name="virt_Ypf3">
+		<inertial>
+			<origin xyz="0 0 0" rpy="0 0 0"/>
+			<mass value="0.001"/>
+			<inertia ixx="0.001" ixy="0" ixz="0" iyy="0.001" iyz="0" izz="0.001"/>
+		</inertial>
+	</link>
+	<joint name="rev_Zpf3" type="revolute">
+		<origin xyz="0 0 1.7320508075688772" rpy="0 0 0"/>
+		<parent link="cable3"/>
+		<child link="virt_Ypf3"/>
+		<axis xyz="0 0 1"/>
+		<limit effort="10000" velocity="0.25"/>
+		<limit damping="0.1"/>
+	</joint>
+	<gazebo>
+		<joint name="rev_Ypf3" type="revolute">
+			<pose>0 0 0 -2.436024 -0.300730 0.780760</pose>
+			<parent>virt_Xpf3</parent>
+			<child>virt_Ypf3</child>
+			<axis>
+				<xyz>0 1 0</xyz>
+				<limit>
+					<effort>10000</effort>
+					<velocity>0.25</velocity>
+				</limit>
+				<dynamics>
+					<damping>0.1</damping>
+				</dynamics>
+			</axis>
+		</joint>
+	</gazebo>
+	<gazebo reference="cable3">
+		<material>Gazebo/Red</material>
+	</gazebo>
+	<gazebo reference="cable3">
+		<material>Gazebo/Red</material>
+	</gazebo>
 	<link name="cable4">
 		<collision>
+			<origin xyz="0 0 -0.06847033160746463" rpy="0 0 0"/>
 			<geometry>
 				<cylinder radius="0.005" length="3.4641016151377544"/>
@@ -400,4 +581,5 @@
 		</visual>
 		<inertial>
+			<origin xyz="0 0 -0.06847033160746463" rpy="0 0 0"/>
 			<geometry>
 				<cylinder radius="0.005" length="3.4641016151377544"/>
@@ -472,4 +654,9 @@
 			</geometry>
 			<material name="${cable_color}"/>
+			<origin xyz="0.150000 0.150000 0.350000" rpy="-1.275355 0.763259 -0.578033"/>
+			<geometry>
+				<box size="0.1 0.1 0.1"/>
+			</geometry>
+			<material name="${cable_color}"/>
 		</visual>
 	</link>
@@ -482,6 +669,45 @@
 		<limit damping="0.1"/>
 	</joint>
+	<link name="virt_Ypf4">
+		<inertial>
+			<origin xyz="0 0 0" rpy="0 0 0"/>
+			<mass value="0.001"/>
+			<inertia ixx="0.001" ixy="0" ixz="0" iyy="0.001" iyz="0" izz="0.001"/>
+		</inertial>
+	</link>
+	<joint name="rev_Zpf4" type="revolute">
+		<origin xyz="0 0 1.7320508075688772" rpy="0 0 0"/>
+		<parent link="cable4"/>
+		<child link="virt_Ypf4"/>
+		<axis xyz="0 0 1"/>
+		<limit effort="10000" velocity="0.25"/>
+		<limit damping="0.1"/>
+	</joint>
+	<gazebo>
+		<joint name="rev_Ypf4" type="revolute">
+			<pose>0 0 0 -1.275355 0.763259 -0.578033</pose>
+			<parent>virt_Xpf4</parent>
+			<child>virt_Ypf4</child>
+			<axis>
+				<xyz>0 1 0</xyz>
+				<limit>
+					<effort>10000</effort>
+					<velocity>0.25</velocity>
+				</limit>
+				<dynamics>
+					<damping>0.1</damping>
+				</dynamics>
+			</axis>
+		</joint>
+	</gazebo>
+	<gazebo reference="cable4">
+		<material>Gazebo/Red</material>
+	</gazebo>
+	<gazebo reference="cable4">
+		<material>Gazebo/Red</material>
+	</gazebo>
 	<link name="cable5">
 		<collision>
+			<origin xyz="0 0 -0.41012040092864877" rpy="0 0 0"/>
 			<geometry>
 				<cylinder radius="0.005" length="3.4641016151377544"/>
@@ -496,4 +722,5 @@
 		</visual>
 		<inertial>
+			<origin xyz="0 0 -0.41012040092864877" rpy="0 0 0"/>
 			<geometry>
 				<cylinder radius="0.005" length="3.4641016151377544"/>
@@ -568,4 +795,9 @@
 			</geometry>
 			<material name="${cable_color}"/>
+			<origin xyz="0.150000 0.450000 0.350000" rpy="1.004067 1.055080 0.619089"/>
+			<geometry>
+				<box size="0.1 0.1 0.1"/>
+			</geometry>
+			<material name="${cable_color}"/>
 		</visual>
 	</link>
@@ -578,6 +810,45 @@
 		<limit damping="0.1"/>
 	</joint>
+	<link name="virt_Ypf5">
+		<inertial>
+			<origin xyz="0 0 0" rpy="0 0 0"/>
+			<mass value="0.001"/>
+			<inertia ixx="0.001" ixy="0" ixz="0" iyy="0.001" iyz="0" izz="0.001"/>
+		</inertial>
+	</link>
+	<joint name="rev_Zpf5" type="revolute">
+		<origin xyz="0 0 1.7320508075688772" rpy="0 0 0"/>
+		<parent link="cable5"/>
+		<child link="virt_Ypf5"/>
+		<axis xyz="0 0 1"/>
+		<limit effort="10000" velocity="0.25"/>
+		<limit damping="0.1"/>
+	</joint>
+	<gazebo>
+		<joint name="rev_Ypf5" type="revolute">
+			<pose>0 0 0 1.004067 1.055080 0.619089</pose>
+			<parent>virt_Xpf5</parent>
+			<child>virt_Ypf5</child>
+			<axis>
+				<xyz>0 1 0</xyz>
+				<limit>
+					<effort>10000</effort>
+					<velocity>0.25</velocity>
+				</limit>
+				<dynamics>
+					<damping>0.1</damping>
+				</dynamics>
+			</axis>
+		</joint>
+	</gazebo>
+	<gazebo reference="cable5">
+		<material>Gazebo/Red</material>
+	</gazebo>
+	<gazebo reference="cable5">
+		<material>Gazebo/Red</material>
+	</gazebo>
 	<link name="cable6">
 		<collision>
+			<origin xyz="0 0 -0.8791147021072782" rpy="0 0 0"/>
 			<geometry>
 				<cylinder radius="0.005" length="3.4641016151377544"/>
@@ -592,4 +863,5 @@
 		</visual>
 		<inertial>
+			<origin xyz="0 0 -0.8791147021072782" rpy="0 0 0"/>
 			<geometry>
 				<cylinder radius="0.005" length="3.4641016151377544"/>
@@ -664,4 +936,9 @@
 			</geometry>
 			<material name="${cable_color}"/>
+			<origin xyz="0.450000 0.450000 0.350000" rpy="1.004067 -0.700803 -0.396004"/>
+			<geometry>
+				<box size="0.1 0.1 0.1"/>
+			</geometry>
+			<material name="${cable_color}"/>
 		</visual>
 	</link>
@@ -674,6 +951,45 @@
 		<limit damping="0.1"/>
 	</joint>
+	<link name="virt_Ypf6">
+		<inertial>
+			<origin xyz="0 0 0" rpy="0 0 0"/>
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